File: V2.0-Full-Bridge/Hardware_Design/ClassDFB/ClassDFB.kicad_sch (KiCad schematic)
At the start: 41 parts, among them J1 OUTPUT, Q1 NMOS, Q2 NMOS, Q3 NMOS, Q4 NMOS, U1 IRS20957S, U2 IRS20957S, U3 LM1117MP-3.3

Commit message: Left side completed on schematic
Parts:
- removed C2: 10u, Package_TO_SOT_SMD:SOT-223-3_TabPin2, symbol Device:C
- removed C3: 100u, symbol Device:C
- removed R10, R19, R20, R6, R7: R, symbol Device:R
- removed R5: 1K, Diode_THT:D_DO-35_SOD27_P7.62mm_Horizontal, symbol Device:R
- removed U3: LM1117MP-3.3, Package_TO_SOT_SMD:SOT-223-3_TabPin2, symbol Regulator_Linear:LM1117MP-3.3
- C4, C7: value C -> 1u
- C5, C6: value C -> 2.2u
- J1: value OUTPUT -> OUTPUT_LEFT
- Q1: footprint Package_DFN_QFN:DHVQFN-16-1EP_2.5x3.5mm_P0.5mm_EP1x2mm -> Lib:TRANS_AON7407
- Q2, Q3, Q4: footprint (none) -> Lib:TRANS_AON7407
- R1, R2: value 22 -> 4.7
- R11: value 68 -> 10k; footprint Diode_THT:D_DO-35_SOD27_P7.62mm_Horizontal -> (none)
- R12: value 680 -> 10k; footprint Diode_THT:D_DO-35_SOD27_P7.62mm_Horizontal -> (none)
- R13: value 1K -> 9k; footprint Diode_THT:D_DO-35_SOD27_P7.62mm_Horizontal -> (none)
- R14: value R -> 9k
- R15, R16: value 22 -> 10k
- R17, R18: value R -> 1k
- R3: value 68 -> 4.7; footprint Diode_THT:D_DO-35_SOD27_P7.62mm_Horizontal -> (none)
- R4: value 680 -> 4.7; footprint Diode_THT:D_DO-35_SOD27_P7.62mm_Horizontal -> (none)
- R8, R9: value R -> 560
Connections:
- net +12V: now also R9.2; no longer R11.1, R14.1, R14.2, R3.1, R8.1, U1.1 (VDD), U2.1 (VDD)
- net GND: now also R11.2, R15.2, R17.2, R18.2; no longer R13.2
- net at C4.1, D1.1 (K), U1.15 (VB): now also R12.1; no longer R18.1
- net at D4.2 (A): now also R16.2, U2.16 (CSH)
- net at Q4.2 (G): now also R4.2; no longer R16.2
- net at U1.16 (CSH): now also D2.2 (A), R12.2; no longer R17.1
- net at U1.6 (VREF): now also R13.1
- net at U1.7 (OCSET): now also R13.2, R17.1
- net at U1.8 (DT): now also R11.1; no longer R4.2
- net at Q3.2 (G): now also R3.2; no longer R15.2
- net at R4.1: now also U2.10 (LO); no longer R3.2
- net at C7.1, D3.1 (K), U2.15 (VB): now also R16.1
- net at U2.14 (HO): now also R3.1; no longer R15.1
- net at R9.1: now also U2.1 (VDD); no longer U2.6 (VREF)
- net at U2.7 (OCSET): now also R14.2, R18.1; no longer R9.2
- new net: R8.1, U1.1 (VDD)
- new net: R14.1, U2.6 (VREF)
- new net: R15.1, U2.8 (DT)
